Commit message: Refactoring

File: jaco_description/urdf/gazebo/jaco.urdf (robot description, URDF)
Before this commit: robot jaco, 12 links, 11 joints
Links:
- removed link base_link
- added link jaco_gripper_link, mass 0.3; collision mesh filename=package://jaco_description/meshes/hand_with_noFinger.stl scale=0.001 0.001 0.001; visual mesh filename=package://jaco_description/meshes/hand_with_noFinger.stl scale=0.001 0.001 0.001
- link jaco_finger_link_1: geometry collision mesh filename=package://jaco_description/meshes/finger.stl scale=1.1 1.1 1.1; visual mesh filename=package://jaco_description/meshes/finger.stl scale=1.1 1.1 1.1
- link jaco_finger_link_2: geometry collision mesh filename=package://jaco_description/meshes/finger.stl scale=1.1 1.1 1.1; visual mesh filename=package://jaco_description/meshes/finger.stl scale=1.1 1.1 1.1
- link jaco_finger_link_3: geometry collision mesh filename=package://jaco_description/meshes/finger.stl scale=1.1 1.1 1.1; visual mesh filename=package://jaco_description/meshes/finger.stl scale=1.1 1.1 1.1
- link jaco_link_6: mass 0.3 -> None; geometry 
Joints:
- removed joint base_joint
- added joint jaco_gripper_attach_joint: type fixed, parent jaco_link_6, child jaco_gripper_link
- joint jaco_gripper_tool_frame_joint: origin xyz=0 0 -0.08 rpy=0.23 -1.570796327 1.570796327 -> xyz=0 0 -0.08 rpy=0.17 -1.570796327 1.570796327; parent jaco_link_6 -> jaco_gripper_link
- joint jaco_joint_1: limit lower=-3.14159265359 upper=3.14159265359 effort=30 velocity=5 -> effort=30 velocity=5; type revolute -> continuous
- joint jaco_joint_2: limit lower=-3.14159265359 upper=3.14159265359 effort=30 velocity=5 -> effort=30 velocity=5; type revolute -> continuous
- joint jaco_joint_3: limit lower=-3.14159265359 upper=3.14159265359 effort=30 velocity=5 -> effort=30 velocity=5; type revolute -> continuous
- joint jaco_joint_4: limit lower=-3.14159265359 upper=3.14159265359 effort=30 velocity=5 -> effort=30 velocity=5; type revolute -> continuous
- joint jaco_joint_5: limit lower=-3.14159265359 upper=3.14159265359 effort=30 velocity=5 -> effort=30 velocity=5; type revolute -> continuous

File: jaco_description/urdf/gazebo/jaco.urdf.xacro (robot description, xacro)
@@ -234,36 +234,13 @@
 		<limit lower="${-PI}" upper="${PI}" effort="30" velocity="5"/>
 	</joint>
-	<link name="jaco_link_6">
-		<inertial>
-			<mass value="0.3"/>
-			<inertia ixx="${inertia}"  ixy="0"  ixz="0" iyy="${inertia}" iyz="0" izz="${inertia}" />
-			<origin/>
-		</inertial>
-		<visual>
-			<material name="JacoGrey" />
-			<origin xyz="0 0 -0.1850" rpy="0 0 -3.1415926535897931"/>
-			<!--<origin xyz="0 0 -0.1850" rpy="0 0 0"/>      -->
-			<geometry>
-				<mesh filename="package://jaco_description/meshes/hand_with_noFinger.stl"
-				scale="0.001 0.001 0.001"/>
-			</geometry>
-		</visual>
-		<collision>
-			<origin xyz="0 0 -0.1850" rpy="0 0 -3.1415926535897931"/>
-			<!--<origin xyz="0 0 -0.1850" rpy="0 0 0"/>-->
-			<geometry>
-				<mesh filename="package://jaco_description/meshes/hand_with_noFinger.stl"
-				scale="0.001 0.001 0.001"/>
-			</geometry>
-		</collision>
-	</link>
-	<gazebo reference="jaco_link_6">
-		<material>Gazebo/Blue</material>
-		<turnGravityOff>true</turnGravityOff>
-	</gazebo>
-     <joint name="jaco_gripper_tool_frame_joint" type="fixed">
+    <link name="jaco_link_6"/>
+    <joint name= "jaco_gripper_attach_joint" type="fixed">
+        <parent link="jaco_link_6"/>
+        <child link="jaco_gripper_link" />
+    </joint>
+    <joint name="jaco_gripper_tool_frame_joint" type="fixed">
       <parent link="jaco_link_6"/>
       <child link="jaco_gripper_tool_frame" />
-      <origin xyz="0 0 -0.08" rpy="0.17 ${-3.141592654/2} ${3.141592654/2}"/>
+      <origin xyz="0 0 -0.07" rpy="0.17 ${-3.141592654/2} ${3.141592654/2}"/>
     </joint>
     <link name="jaco_gripper_tool_frame">
@@ -272,4 +249,32 @@
          arm part attached to this link -->
   </link>
+	<link name="jaco_gripper_link">
+		<inertial>
+			<mass value="0.3"/>
+			<inertia ixx="${inertia}"  ixy="0"  ixz="0" iyy="${inertia}" iyz="0" izz="${inertia}" />
+			<origin/>
+		</inertial>
+		<visual>
+			<material name="JacoGrey" />
+			<origin xyz="0 0 -0.1850" rpy="0 0 -3.1415926535897931"/>
+			<!--<origin xyz="0 0 -0.1850" rpy="0 0 0"/>      -->
+			<geometry>
+				<mesh filename="package://jaco_description/meshes/hand_with_noFinger.stl"
+				scale="0.001 0.001 0.001"/>
+			</geometry>
+		</visual>
+		<collision>
+			<origin xyz="0 0 -0.1850" rpy="0 0 -3.1415926535897931"/>
+			<!--<origin xyz="0 0 -0.1850" rpy="0 0 0"/>-->
+			<geometry>
+				<mesh filename="package://jaco_description/meshes/hand_with_noFinger.stl"
+				scale="0.001 0.001 0.001"/>
+			</geometry>
+		</collision>
+	</link>
+	<gazebo reference="jaco_link_6">
+		<material>Gazebo/Blue</material>
+		<turnGravityOff>true</turnGravityOff>
+	</gazebo>
 	<!-- first finger joint & link -->
    	<joint name="jaco_finger_joint_1" type="revolute">
