Commit message: Set joint types to continuous instead of -PI .. PI

File: jaco_description/urdf/gazebo/jaco.urdf.xacro (robot description, xacro)
@@ -54,5 +54,5 @@
 	</gazebo>
 	<!-- First revolute joint & link -->
-	<joint name="jaco_joint_1" type="revolute">
+	<joint name="jaco_joint_1" type="continuous">
 		<!--origin xyz="0 0 0.2102" rpy="0 0 0"/-->
         	<origin xyz="0 0 0.2725" rpy="0 0 0"/>
@@ -60,5 +60,5 @@
 		<parent link="jaco_base_link"/>
 		<child link="jaco_link_1"/>
-		<limit lower="${-PI}" upper="${PI}" effort="30" velocity="5"/>
+		<limit effort="30" velocity="5"/>
 	</joint>
 	<link name="jaco_link_1">
@@ -89,10 +89,10 @@
 	</gazebo>
 	<!-- Second revolute joint & link -->
-	<joint name="jaco_joint_2" type="revolute">
+	<joint name="jaco_joint_2" type="continuous">
 		<origin xyz="0 0 0" rpy="-1.570796327 0 0"/>
 		<axis xyz="0 0 1"/>
 		<parent link="jaco_link_1"/>
 		<child link="jaco_link_2"/>
-		<limit lower="${-PI}" upper="${PI}" effort="30" velocity="5"/>
+		<limit effort="30" velocity="5"/>
 	</joint>
 	<link name="jaco_link_2">
@@ -123,10 +123,10 @@
 	</gazebo>
 	<!-- Third revolute joint & link -->
-	<joint name="jaco_joint_3" type="revolute">
+	<joint name="jaco_joint_3" type="continuous">
 		<origin xyz="0.4100 0 0.012" rpy="0 0 0"/>
 		<axis xyz="0 0 -1"/>
 		<parent link="jaco_link_2"/>
 		<child link="jaco_link_3"/>
-		<limit lower="${-PI}" upper="${PI}" effort="30" velocity="5"/>
+		<limit effort="30" velocity="5"/>
 	</joint>
 	<link name="jaco_link_3">
@@ -157,10 +157,10 @@
 	</gazebo>
 	<!-- Fourth revolute joint & link -->
-	<joint name="jaco_joint_4" type="revolute">
+	<joint name="jaco_joint_4" type="continuous">
 		<origin xyz="0 0.24927682300748782 0 " rpy="-1.570796327 0 0"/>
 		<axis xyz="0 0 -1"/>
 		<parent link="jaco_link_3"/>
 		<child link="jaco_link_4"/>
-		<limit lower="${-PI}" upper="${PI}" effort="30" velocity="5"/>
+		<limit effort="30" velocity="5"/>
 	</joint>
 	<link name="jaco_link_4">
@@ -191,10 +191,10 @@
 	</gazebo>
 	<!-- Fifth revolute joint & link -->
-	<joint name="jaco_joint_5" type="revolute">
+	<joint name="jaco_joint_5" type="continuous">
 		<origin xyz="0 -0.069262292 0.048497979" rpy="0.959931089 0 0"/>
 		<axis xyz="0 0 -1"/>
 		<parent link="jaco_link_4"/>
 		<child link="jaco_link_5"/>
-		<limit lower="${-PI}" upper="${PI}" effort="30" velocity="5"/>
+		<limit effort="30" velocity="5"/>
 	</joint>
 	<link name="jaco_link_5">
@@ -291,5 +291,5 @@
           <geometry>
             <mesh filename="package://jaco_description/meshes/finger.stl"
-                scale="1 1 1"/>
+                scale="1.1 1.1 1.1"/>
           </geometry>
     </visual>
@@ -298,5 +298,5 @@
 	<geometry>
         <mesh filename="package://jaco_description/meshes/finger.stl"
-                scale="1 1 1"/>
+                scale="1.1 1.1 1.1"/>
 	</geometry>
 	</collision>
@@ -325,5 +325,5 @@
           <geometry>
             <mesh filename="package://jaco_description/meshes/finger.stl"
-                scale="1 1 1"/>
+                scale="1.1 1.1 1.1"/>
           </geometry>
         </visual>
@@ -332,5 +332,5 @@
 	<geometry>
             <mesh filename="package://jaco_description/meshes/finger.stl"
-                scale="1 1 1"/>
+                scale="1.1 1.1 1.1"/>
 	</geometry>
 	</collision>
@@ -359,5 +359,5 @@
           <geometry>
             <mesh filename="package://jaco_description/meshes/finger.stl"
-                scale="1 1 1"/>
+                scale="1.1 1.1 1.1"/>
           </geometry>
         </visual>
@@ -366,5 +366,5 @@
 	<geometry>
             <mesh filename="package://jaco_description/meshes/finger.stl"
-                scale="1 1 1"/>
+                scale="1.1 1.1 1.1"/>
 	</geometry>
 	</collision>

Commit message: Improved jaco_gripper_tool frame orientation to match the real upright position of the gripper

File: jaco_description/urdf/gazebo/jaco.urdf.xacro (robot description, xacro)
@@ -265,5 +265,5 @@
       <parent link="jaco_link_6"/>
       <child link="jaco_gripper_tool_frame" />
-      <origin xyz="0 0 -0.08" rpy="0.23 ${-3.141592654/2} ${3.141592654/2}"/>
+      <origin xyz="0 0 -0.08" rpy="0.17 ${-3.141592654/2} ${3.141592654/2}"/>
     </joint>
     <link name="jaco_gripper_tool_frame">

Commit message: Corrected fingersize, adapted home position, new calibrate launch files and alvar launch files

File: jaco_description/urdf/gazebo/jaco.urdf.xacro (robot description, xacro)
@@ -1,21 +1,20 @@
-<?xml version="1.0"?>
-<robot name="jaco"
-  xmlns:xacro="http://ros.org/wiki/xacro">
- <xacro:property name="inertia" value="1" />
-  <xacro:property name="finger_inertia" value="1" />
-  <xacro:property name="PI" value="3.1415926535897931" />
-	<gazebo>
-    <plugin name="gazebo_ros_controller_manager" filename="libgazebo_ros_controller_manager.so">
-      <alwaysOn>true</alwaysOn>
-		<updateRate>1000.0</updateRate>
-		<robotParam>robot_description</robotParam>
-    </plugin>
-	</gazebo>
-	<xacro:include filename="$(find jaco_description)/urdf/gazebo/jaco.gazebo.xacro" />
-	<xacro:include filename="$(find jaco_description)/urdf/gazebo/jaco.transmissions.xacro" />
-	<material name="JacoGrey">
-	<color rgba="0.2 0.2 0.9 1.0"/>
-	</material>
-	<!--
+<?xml version="1.0" encoding="UTF-8"?>
+<robot name="jaco" xmlns:xacro="http://ros.org/wiki/xacro">
+    <xacro:property name="inertia" value="1"/>
+    <xacro:property name="finger_inertia" value="1"/>
+    <xacro:property name="PI" value="3.1415926535897931"/>
+    <gazebo>
+        <plugin filename="libgazebo_ros_controller_manager.so" name="gazebo_ros_controller_manager">
+            <alwaysOn>true</alwaysOn>
+            <updateRate>1000.0</updateRate>
+            <robotParam>robot_description</robotParam>
+        </plugin>
+    </gazebo>
+    <xacro:include filename="$(find jaco_description)/urdf/gazebo/jaco.gazebo.xacro"/>
+    <xacro:include filename="$(find jaco_description)/urdf/gazebo/jaco.transmissions.xacro"/>
+    <material name="JacoGrey">
+        <color rgba="0.2 0.2 0.9 1.0"/>
+    </material>
+    <!--
 	<link name="world"/>
 	<joint name="base_block_joint" type="fixed">
@@ -25,357 +24,383 @@
 	</joint>
  -->
-	<!-- The base joint & link -->
-	<link name="jaco_base_link">
-		<inertial>
-			<mass value="1" />
-			<!--origin xyz="0 0 -0.0525" rpy="0 0 0"/-->
-          		<origin xyz="0 0 0.0" rpy="0 0 0"/>
-			<inertia ixx="${inertia}"  ixy="0"  ixz="0" iyy="${inertia}" iyz="0" izz="${inertia}" />
-		</inertial>
-		<visual>
-			<material name="JacoGrey" />
-			<!--origin xyz="0 0 -0.0525" rpy="0 0 0"/-->
-			<geometry>
-				<mesh filename="package://jaco_description/meshes/joint_1.stl"
-				scale="0.001 0.001 0.001"/>
-			</geometry>
-		</visual>
-		<collision>
-			<!--origin xyz="0 0 -0.0525" rpy="0 0 0"/-->
-			<geometry>
-				<mesh filename="package://jaco_description/meshes/joint_1.stl"
-				scale="0.001 0.001 0.001"/>
-			</geometry>
-		</collision>
-	</link>
-	<gazebo reference="jaco_base_link">
-		<material>Gazebo/Yellow</material>
-		<turnGravityOff>true</turnGravityOff>
-	</gazebo>
-	<!-- First revolute joint & link -->
-	<joint name="jaco_joint_1" type="continuous">
-		<!--origin xyz="0 0 0.2102" rpy="0 0 0"/-->
-        	<origin xyz="0 0 0.2725" rpy="0 0 0"/>
-		<axis xyz="0 0 -1" rpy="0 0 0"/>
-		<parent link="jaco_base_link"/>
-		<child link="jaco_link_1"/>
-		<limit effort="30" velocity="5"/>
-	</joint>
-	<link name="jaco_link_1">
-		<inertial>
-			<mass value="1" />
-			<inertia ixx="${inertia}"  ixy="0"  ixz="0" iyy="${inertia}" iyz="0" izz="${inertia}" />
-			<origin/>
-		</inertial>
-		<visual>
-			<material name="JacoGrey" />
-			<origin xyz="0 0 -0.12" rpy="0 0 -1.570796327"/>
-			<geometry>
-				<mesh filename="package://jaco_description/meshes/joint_2.stl"
-				scale="0.001 0.001 0.001"/>
-			</geometry>
-		</visual>
-		<collision>
-			<origin xyz="0 0 -0.12" rpy="0 0 -1.570796327"/>
-			<geometry>
-				<mesh filename="package://jaco_description/meshes/joint_2.stl"
-				scale="0.001 0.001 0.001"/>
-			</geometry>
-		</collision>
-	</link>
-	<gazebo reference="jaco_link_1">
-		<material>Gazebo/Red</material>
-		<turnGravityOff>true</turnGravityOff>
-	</gazebo>
-	<!-- Second revolute joint & link -->
-	<joint name="jaco_joint_2" type="continuous">
-		<origin xyz="0 0 0" rpy="-1.570796327 0 0"/>
-		<axis xyz="0 0 1"/>
-		<parent link="jaco_link_1"/>
-		<child link="jaco_link_2"/>
-		<limit effort="30" velocity="5"/>
-	</joint>
-	<link name="jaco_link_2">
-		<inertial>
-			<mass value="1" />
-			<inertia ixx="${inertia}"  ixy="0"  ixz="0" iyy="${inertia}" iyz="0" izz="${inertia}" />
-			<origin/>
-		</inertial>
-		<visual>
-			<material name="JacoGrey" />
-			<origin xyz="0 0 0.015" rpy="0 1.570796327 0"/>
-			<geometry>
-				<mesh filename="package://jaco_description/meshes/joint_3.stl"
-				scale="0.001 0.001 0.001"/>
-			</geometry>
-		</visual>
-		<collision>
-			<origin xyz="0 0 0.015" rpy="0 1.570796327 0"/>
-			<geometry>
-				<mesh filename="package://jaco_description/meshes/joint_3.stl"
-				scale="0.001 0.001 0.001"/>
-			</geometry>
-		</collision>
-	</link>
-	<gazebo reference="jaco_link_2">
-		<material>Gazebo/Blue</material>
-		<turnGravityOff>true</turnGravityOff>
-	</gazebo>
-	<!-- Third revolute joint & link -->
-	<joint name="jaco_joint_3" type="continuous">
-		<origin xyz="0.4100 0 0.012" rpy="0 0 0"/>
-		<axis xyz="0 0 -1"/>
-		<parent link="jaco_link_2"/>
-		<child link="jaco_link_3"/>
-		<limit effort="30" velocity="5"/>
-	</joint>
-	<link name="jaco_link_3">
-		<inertial>
-			<mass value="1" />
-			<inertia ixx="${inertia}"  ixy="0"  ixz="0" iyy="${inertia}" iyz="0" izz="${inertia}" />
-			<origin/>
-		</inertial>
-		<visual>
-			<material name="JacoGrey" />
-			<origin xyz="0 0 -0.012" rpy="0 1.570796327 1.570796327"/>
-			<geometry>
-				<mesh filename="package://jaco_description/meshes/joint_4.stl"
-				scale="1.000 1.000 1.000"/>
-			</geometry>
-		</visual>
-		<collision>
-			<origin xyz="0 0 -0.012" rpy="0 1.570796327 1.570796327"/>
-			<geometry>
-				<mesh filename="package://jaco_description/meshes/joint_4.stl"
-				scale="1.000 1.000 1.000"/>
-			</geometry>
-		</collision>
-	</link>
-	<gazebo reference="jaco_link_3">
-		<material>Gazebo/Red</material>
-		<turnGravityOff>true</turnGravityOff>
-	</gazebo>
-	<!-- Fourth revolute joint & link -->
-	<joint name="jaco_joint_4" type="continuous">
-		<origin xyz="0 0.24927682300748782 0 " rpy="-1.570796327 0 0"/>
-		<axis xyz="0 0 -1"/>
-		<parent link="jaco_link_3"/>
-		<child link="jaco_link_4"/>
-		<limit effort="30" velocity="5"/>
-	</joint>
-	<link name="jaco_link_4">
-		<inertial>
-			<mass value="1" />
-			<inertia ixx="${inertia}"  ixy="0"  ixz="0" iyy="${inertia}" iyz="0" izz="${inertia}" />
-			<origin/>
-		</inertial>
-		<visual>
-			<material name="JacoGrey" />
-			<origin xyz="0 0 -0.042276823" rpy="0 0 -1.570796327"/>
-			<geometry>
-				<mesh filename="package://jaco_description/meshes/joint_5.stl"
-				scale="0.001 0.001 0.001"/>
-			</geometry>
-		</visual>
-		<collision>
-			<origin xyz="0 0 -0.042276823" rpy="0 0 -1.570796327"/>
-			<geometry>
-				<mesh filename="package://jaco_description/meshes/joint_5.stl"
-				scale="0.001 0.001 0.001"/>
-			</geometry>
-		</collision>
-	</link>
-	<gazebo reference="jaco_link_4">
-		<material>Gazebo/Blue</material>
-		<turnGravityOff>true</turnGravityOff>
-	</gazebo>
-	<!-- Fifth revolute joint & link -->
-	<joint name="jaco_joint_5" type="continuous">
-		<origin xyz="0 -0.069262292 0.048497979" rpy="0.959931089 0 0"/>
-		<axis xyz="0 0 -1"/>
-		<parent link="jaco_link_4"/>
-		<child link="jaco_link_5"/>
-		<limit effort="30" velocity="5"/>
-	</joint>
-	<link name="jaco_link_5">
-		<inertial>
-			<mass value="1.0"/>
-			<inertia ixx="${inertia}"  ixy="0"  ixz="0" iyy="${inertia}" iyz="0" izz="${inertia}" />
-			<origin/>
-		</inertial>
-		<visual>
-			<material name="JacoGrey" />
-			<origin xyz="0 0 -0.042276823" rpy="0 -0.959931089 1.570796327"/>
-			<geometry>
-				<mesh filename="package://jaco_description/meshes/joint_6.stl"
-				scale="0.001 0.001 0.001"/>
-			</geometry>
-		</visual>
-		<collision>
-			<origin xyz="0 0 -0.042276823" rpy="0 -0.959931089 1.570796327"/>
-			<geometry>
-				<mesh filename="package://jaco_description/meshes/joint_6.stl"
-				scale="0.001 0.001 0.001"/>
-			</geometry>
-		</collision>
-	</link>
-	<gazebo reference="jaco_link_5">
-		<material>Gazebo/Red</material>
-		<turnGravityOff>true</turnGravityOff>
-	</gazebo>
-	<!-- Sixth revolute joint & link -->
-	<joint name="jaco_joint_6" type="revolute">
-		<!--origin xyz="0 -0.186174274 0.13036063" rpy="0.959931089 0 0"/-->
-		<origin xyz="0 -0.186174274 0.13036063" rpy="-0.959931089 0 3.1415926535897931"/>
-		<!--<origin xyz="0 0 0" rpy="0 0 -3.14"/>-->
-		<axis xyz="0 0 -1"/>
-		<parent link="jaco_link_5"/>
-		<child link="jaco_link_6"/>
-		<limit lower="${-PI}" upper="${PI}" effort="30" velocity="5"/>
-	</joint>
+    <!-- The base joint & link -->
+    <link name="jaco_base_link">
+        <inertial>
+            <mass value="1"/>
+            <!--origin xyz="0 0 -0.0525" rpy="0 0 0"/-->
+            <origin rpy="0 0 0" xyz="0 0 0.0"/>
+            <inertia ixx="${inertia}" ixy="0" ixz="0" iyy="${inertia}"
+                iyz="0" izz="${inertia}"/>
+        </inertial>
+        <visual>
+            <material name="JacoGrey"/>
+            <!--origin xyz="0 0 -0.0525" rpy="0 0 0"/-->
+            <geometry>
+                <mesh
+                    filename="package://jaco_description/meshes/joint_1.stl" scale="0.001 0.001 0.001"/>
+            </geometry>
+        </visual>
+        <collision>
+            <!--origin xyz="0 0 -0.0525" rpy="0 0 0"/-->
+            <geometry>
+                <mesh
+                    filename="package://jaco_description/meshes/joint_1.stl" scale="0.001 0.001 0.001"/>
+            </geometry>
+        </collision>
+    </link>
+    <gazebo reference="jaco_base_link">
+        <material>Gazebo/Yellow</material>
+        <turnGravityOff>true</turnGravityOff>
+    </gazebo>
+    <!-- First revolute joint & link -->
+    <joint name="jaco_joint_1" type="continuous">
+        <!--origin xyz="0 0 0.2102" rpy="0 0 0"/-->
+        <origin rpy="0 0 0" xyz="0 0 0.2725"/>
+        <axis rpy="0 0 0" xyz="0 0 -1"/>
+        <parent link="jaco_base_link"/>
+        <child link="jaco_link_1"/>
+        <limit effort="30" velocity="5"/>
+    </joint>
+    <link name="jaco_link_1">
+        <inertial>
+            <mass value="1"/>
+            <inertia ixx="${inertia}" ixy="0" ixz="0" iyy="${inertia}"
+                iyz="0" izz="${inertia}"/>
+            <origin/>
+        </inertial>
+        <visual>
+            <material name="JacoGrey"/>
+            <origin rpy="0 0 -1.570796327" xyz="0 0 -0.12"/>
+            <geometry>
+                <mesh
+                    filename="package://jaco_description/meshes/joint_2.stl" scale="0.001 0.001 0.001"/>
+            </geometry>
+        </visual>
+        <collision>
+            <origin rpy="0 0 -1.570796327" xyz="0 0 -0.12"/>
+            <geometry>
+                <mesh
+                    filename="package://jaco_description/meshes/joint_2.stl" scale="0.001 0.001 0.001"/>
+            </geometry>
+        </collision>
+    </link>
+    <gazebo reference="jaco_link_1">
+        <material>Gazebo/Red</material>
+        <turnGravityOff>true</turnGravityOff>
+    </gazebo>
+    <!-- Second revolute joint & link -->
+    <joint name="jaco_joint_2" type="continuous">
+        <origin rpy="-1.570796327 0 0" xyz="0 0 0"/>
+        <axis xyz="0 0 1"/>
+        <parent link="jaco_link_1"/>
+        <child link="jaco_link_2"/>
+        <limit effort="30" velocity="5"/>
+    </joint>
+    <link name="jaco_link_2">
+        <inertial>
+            <mass value="1"/>
+            <inertia ixx="${inertia}" ixy="0" ixz="0" iyy="${inertia}"
+                iyz="0" izz="${inertia}"/>
+            <origin/>
+        </inertial>
+        <visual>
+            <material name="JacoGrey"/>
+            <origin rpy="0 1.570796327 0" xyz="0 0 0.015"/>
+            <geometry>
+                <mesh
+                    filename="package://jaco_description/meshes/joint_3.stl" scale="0.001 0.001 0.001"/>
+            </geometry>
+        </visual>
+        <collision>
+            <origin rpy="0 1.570796327 0" xyz="0 0 0.015"/>
+            <geometry>
+                <mesh
+                    filename="package://jaco_description/meshes/joint_3.stl" scale="0.001 0.001 0.001"/>
+            </geometry>
+        </collision>
+    </link>
+    <gazebo reference="jaco_link_2">
+        <material>Gazebo/Blue</material>
+        <turnGravityOff>true</turnGravityOff>
+    </gazebo>
+    <!-- Third revolute joint & link -->
+    <joint name="jaco_joint_3" type="continuous">
+        <origin rpy="0 0 0" xyz="0.4100 0 0.012"/>
+        <axis xyz="0 0 -1"/>
+        <parent link="jaco_link_2"/>
+        <child link="jaco_link_3"/>
+        <limit effort="30" velocity="5"/>
+    </joint>
+    <link name="jaco_link_3">
+        <inertial>
+            <mass value="1"/>
+            <inertia ixx="${inertia}" ixy="0" ixz="0" iyy="${inertia}"
+                iyz="0" izz="${inertia}"/>
+            <origin/>
+        </inertial>
+        <visual>
+            <material name="JacoGrey"/>
+            <origin rpy="0 1.570796327 1.570796327" xyz="0 0 -0.012"/>
+            <geometry>
+                <mesh
+                    filename="package://jaco_description/meshes/joint_4.stl" scale="1.000 1.000 1.000"/>
+            </geometry>
+        </visual>
+        <collision>
+            <origin rpy="0 1.570796327 1.570796327" xyz="0 0 -0.012"/>
+            <geometry>
+                <mesh
+                    filename="package://jaco_description/meshes/joint_4.stl" scale="1.000 1.000 1.000"/>
+            </geometry>
+        </collision>
+    </link>
+    <gazebo reference="jaco_link_3">
+        <material>Gazebo/Red</material>
+        <turnGravityOff>true</turnGravityOff>
+    </gazebo>
+    <!-- Fourth revolute joint & link -->
+    <joint name="jaco_joint_4" type="continuous">
+        <origin rpy="-1.570796327 0 0" xyz="0 0.24927682300748782 0 "/>
+        <axis xyz="0 0 -1"/>
+        <parent link="jaco_link_3"/>
+        <child link="jaco_link_4"/>
+        <limit effort="30" velocity="5"/>
+    </joint>
+    <link name="jaco_link_4">
+        <inertial>
+            <mass value="1"/>
+            <inertia ixx="${inertia}" ixy="0" ixz="0" iyy="${inertia}"
+                iyz="0" izz="${inertia}"/>
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
Commit message: urdf update

File: jaco_description/urdf/gazebo/jaco.urdf.xacro (robot description, xacro)
@@ -53,4 +53,26 @@
         <turnGravityOff>true</turnGravityOff>
     </gazebo>
+    <joint name="jaco_base_cabels_joint" type="fixed">
+    <parent link="jaco_base_link"/>
+    <child link="cabels"/>
+    <origin xyz="0 0.06 0.05"/>
+    </joint>
+    <link name="cabels">
+    <visual>
+      <origin xyz="0 0 0" rpy="0 0 0" />
+      <geometry>
+        <box size="0.08 0.09 0.2" />
+      </geometry>
+      <material name="black">
+        <color rgba="1 1 1 1"/>
+      </material>
+    </visual>
+    <collision>
+      <origin xyz="0 0 0" rpy="0 0 0" />
+      <geometry>
+        <box size="0.1 0.1 0.2" />
+      </geometry>
+    </collision>
+    </link>
     <!-- First revolute joint & link -->
     <joint name="jaco_joint_1" type="continuous">

Commit message: Added joint limits to jaco joint 2

File: jaco_description/urdf/gazebo/jaco.urdf.xacro (robot description, xacro)
@@ -112,10 +112,10 @@
     </gazebo>
     <!-- Second revolute joint & link -->
-    <joint name="jaco_joint_2" type="continuous">
+    <joint name="jaco_joint_2" type="revolute">
         <origin rpy="-1.570796327 0 0" xyz="0 0 0"/>
         <axis xyz="0 0 1"/>
         <parent link="jaco_link_1"/>
         <child link="jaco_link_2"/>
-        <limit effort="30" velocity="5"/>
+        <limit effort="30" lower="${-PI+PI/8}" upper="${PI/8}" velocity="5"/>
     </joint>
     <link name="jaco_link_2">
